Commit message: moved secondary robot description from fork to master

File: src/mcl/models/primary_robot.urdf.xacro (robot description, xacro)
@@ -145,5 +145,5 @@
       <origin xyz="0 0 0" rpy="0 0 0"/>
       <geometry>
-	<mesh filename="package://mcl/models/apriltag/ar_tag_2.dae" scale="0.5 0.5 0.5"/>
+	<mesh filename="package://mcl/models/apriltag/ar_tag_2.dae" scale="1 1 1"/>
       </geometry>
     </visual>

Commit message: multi-robot sim

File: src/mcl/models/primary_robot.urdf.xacro (robot description, xacro)
@@ -113,4 +113,6 @@
   </joint>
   <link name="imu_link"/>
+  <!-- Primary robot has no scanner -->
+  <!--
   <joint name="scan_joint" type="fixed">
     <parent link="base_link"/>
@@ -139,5 +141,5 @@
                izz="0.001" />
     </inertial>\`
-  </link>
+  </link> -->
   <!-- April Tag -->
   <link name="april_tag">
@@ -150,7 +152,7 @@
   </link>
   <joint name="apriltag_joint" type="fixed">
-    <parent link="base_scan"/>
+    <parent link="base_link"/>
     <child link="april_tag"/>
-    <origin xyz="0 0 0.034" rpy="0 0 0"/>
+    <origin xyz="0 0 0.206" rpy="0 0 0"/>
   </joint>
 </robot>

Commit message: Apriltag detection integration

File: src/mcl/models/primary_robot.urdf.xacro (robot description, xacro)
@@ -147,5 +147,5 @@
       <origin xyz="0 0 0" rpy="0 0 0"/>
       <geometry>
-	<mesh filename="package://mcl/models/apriltag/ar_tag_2.dae" scale="1 1 1"/>
+	<mesh filename="package://mcl/models/apriltag/four_faces.dae" scale="1 1 1"/>
       </geometry>
     </visual>

Commit message: apriltag tuning

File: src/mcl/models/primary_robot.urdf.xacro (robot description, xacro)
@@ -147,5 +147,5 @@
       <origin xyz="0 0 0" rpy="0 0 0"/>
       <geometry>
-	<mesh filename="package://mcl/models/apriltag/four_faces.dae" scale="1 1 1"/>
+	      <mesh filename="package://mcl/models/apriltag/four_faces.dae" scale="2 2 2"/>
       </geometry>
     </visual>
